Commit message: first commit

File: VEDANT - 211156/src/m2wr_description/urdf/m2wr.xacro (robot description, xacro)
@@ -1,9 +1,9 @@
 <?xml version="1.0" ?>
 <robot name="m2wr" xmlns:xacro="http://www.ros.org/wiki/xacro">
-  <xacro:include filename="$(find m2wr_description)/urdf/materials.xacro"/>
-  <xacro:include filename="$(find m2wr_description)/urdf/m2wr.gazebo"/>
-  <xacro:include filename="$(find m2wr_description)/urdf/macros.xacro"/>
+  <xacro:include filename="$(find m2wr_description)/urdf/materials.xacro" />
+  <xacro:include filename="$(find m2wr_description)/urdf/m2wr.gazebo" />
+  <xacro:include filename="$(find m2wr_description)/urdf/macros.xacro" />
+  <!-- Links -->
   <link name="link_chassis">
-    <!-- pose and inertial -->
     <pose>0 0 0.1 0 0 0</pose>
     <inertial>
@@ -12,5 +12,4 @@
       <inertia ixx="0.0395416666667" ixy="0" ixz="0" iyy="0.106208333333" iyz="0" izz="0.106208333333"/>
     </inertial>
-    <!-- body -->
     <collision name="collision_chassis">
       <geometry>
@@ -25,5 +24,4 @@
       <material name="blue"/>
     </visual>
-    <!-- caster front -->
     <collision name="caster_front_collision">
       <origin rpy=" 0 0 0" xyz="0.35 0 -0.05"/>
@@ -69,12 +67,110 @@
     </collision>
   </link>
-  <joint name="joint_sensor_laser" type="fixed">
-    <origin xyz="0.15 0 0.05" rpy="0 0 0"/>
-    <parent link="link_chassis"/>
-    <child link="sensor_laser"/>
-  </joint>
-  <xacro:link_wheel name="link_right_wheel"/>
-  <xacro:joint_wheel name="joint_right_wheel" child="link_right_wheel" origin_xyz="-0.05 0.15 0"/>
-  <xacro:link_wheel name="link_left_wheel"/>
-  <xacro:joint_wheel name="joint_left_wheel" child="link_left_wheel" origin_xyz="-0.05 -0.15 0"/>
+<link name="camera_link_rear">
+  <visual>
+    <origin xyz="0 0 0" rpy="0 0 0"/>
+    <geometry>
+      <box size="0.015 0.130 0.022"/>
+    </geometry>
+  </visual>
+  <collision>
+    <origin xyz="0 0 0" rpy="0 0 0"/>
+    <geometry>
+      <box size="0.015 0.130 0.022"/>
+    </geometry>
+  </collision>
+  <inertial>
+    <origin xyz="0 0 0" rpy="0 0 0"/>
+    <mass value="0.035"/>
+    <inertia ixx="0.001"  ixy="0"  ixz="0" iyy="0.001" iyz="0" izz="0.001" />
+  </inertial>
+</link>
+<link name="camera_link_front1">
+  <visual>
+    <origin xyz="0 0 0" rpy="0 0 0"/>
+    <geometry>
+      <box size="0.015 0.130 0.022"/>
+    </geometry>
+  </visual>
+  <collision>
+    <origin xyz="0 0 0" rpy="0 0 0"/>
+    <geometry>
+      <box size="0.015 0.130 0.022"/>
+    </geometry>
+  </collision>
+  <inertial>
+    <origin xyz="0 0 0" rpy="0 0 0"/>
+    <mass value="0.035"/>
+    <inertia ixx="0.001"  ixy="0"  ixz="0" iyy="0.001" iyz="0" izz="0.001" />
+  </inertial>
+</link>
+<link name="camera_link_front2">
+  <visual>
+    <origin xyz="0 0 0" rpy="0 0 0"/>
+    <geometry>
+      <box size="0.015 0.130 0.022"/>
+    </geometry>
+  </visual>
+  <collision>
+    <origin xyz="0 0 0" rpy="0 0 0"/>
+    <geometry>
+      <box size="0.015 0.130 0.022"/>
+    </geometry>
+  </collision>
+  <inertial>
+    <origin xyz="0 0 0" rpy="0 0 0"/>
+    <mass value="0.035"/>
+    <inertia ixx="0.001"  ixy="0"  ixz="0" iyy="0.001" iyz="0" izz="0.001" />
+  </inertial>
+</link>
+<link name="imu_link">
+    <inertial>
+      <origin xyz="0 0 0" rpy="0 0 0" />
+      <mass value="1" />
+      <xacro:cylinder_inertia mass="1" r="0.025" l="0.05" />
+    </inertial>
+    <visual>
+      <origin xyz="0 0 0" rpy="0 0 0" />
+      <geometry>
+        <cylinder radius="0.025" length="0.05"/>
+      </geometry>
+      <material name="black" />
+    </visual>
+    <collision>
+      <origin xyz="0 0 0" rpy="0 0 0"/>
+      <geometry>
+        <cylinder radius="0.025" length="0.05"/>
+      </geometry>
+    </collision>
+  </link>
+<!-- Joints -->
+<joint name="joint_imu_link" type="fixed">
+  <origin xyz="0 0 0.05" rpy="0 0 0"/>
+  <parent link="link_chassis"/>
+  <child link="imu_link"/>
+</joint>
+<joint name="camera_joint_rear" type="fixed">
+  <parent link="link_chassis"/>
+  <child link="camera_link_rear"/>
+  <origin xyz="-0.2 0 0.05" rpy="0 0 3.1416"/>
+</joint>
+<joint name="camera_joint_front1" type="fixed">
+  <parent link="link_chassis"/>
+  <child link="camera_link_front1"/>
+  <origin xyz="0.215 0.1 0.05" rpy="0 0 0.3927"/>
+</joint>
+<joint name="camera_joint_front2" type="fixed">
+  <parent link="link_chassis"/>
+  <child link="camera_link_front2"/>
+  <origin xyz="0.215 -0.1 0.05" rpy="0 0 -0.3927"/>
+</joint>
+<joint name="joint_sensor_laser" type="fixed">
+  <origin xyz="0.15 0 0.05" rpy="0 0 0"/>
+  <parent link="link_chassis"/>
+  <child link="sensor_laser"/>
+</joint>
+  <xacro:link_wheel name="link_right_wheel" />
+  <xacro:joint_wheel name="joint_right_wheel" child="link_right_wheel" origin_xyz="-0.05 0.20 0" />
+  <xacro:link_wheel name="link_left_wheel" />
+  <xacro:joint_wheel name="joint_left_wheel" child="link_left_wheel" origin_xyz="-0.05 -0.20 0" />
 </robot>
